File: board/SuperFeed.sch (EAGLE design)
At the start: 16 parts

Commit message: Reducing amount of different hole sizes
Parts:
- R2, R3, R4, R5: device SuperFeed:R-US_0207/15 -> SuperFeed:R-US_0207/10
Changed lines of the file:
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@@
 <part name="R1" library="SuperFeed" deviceset="R-TRIMM" device="T93YA"/>
 <part name="+3V2" library="SuperFeed" deviceset="+3V3" device=""/>
-<part name="R2" library="SuperFeed" deviceset="R-US_" device="0207/15" value="10k"/>
-<part name="R3" library="SuperFeed" deviceset="R-US_" device="0207/15" value="10k"/>
-<part name="R4" library="SuperFeed" deviceset="R-US_" device="0207/15" value="10k"/>
-<part name="R5" library="SuperFeed" deviceset="R-US_" device="0207/15" value="10k"/>
+<part name="R2" library="SuperFeed" deviceset="R-US_" device="0207/10" value="10k"/>
+<part name="R3" library="SuperFeed" deviceset="R-US_" device="0207/10" value="10k"/>
+<part name="R4" library="SuperFeed" deviceset="R-US_" device="0207/10" value="10k"/>
+<part name="R5" library="SuperFeed" deviceset="R-US_" device="0207/10" value="10k"/>
 <part name="P+5" library="SuperFeed" deviceset="+5V" device=""/>
 <part name="EXTBTN" library="SuperFeed" deviceset="MA05-1W" device=""/>
